File: catchrobo2023_Controller/catchrobo2023_Controller.kicad_sch (KiCad schematic)
At the start: 7 parts

Commit message: MDを修正
Connections:
- net Emergency_N renamed +3.3V
- net +3.3V: now also J?.1 (Pin_1); no longer J?.2 (Pin_2)
- net Emergency_P renamed Emergency
- net Emergency: now also J?.2 (Pin_2); no longer J?.1 (Pin_1)
Changed lines of the file:
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@@
     (effects (font (size 1.27 1.27)) (justify left bottom))
   )
-  (label "Emergency_P" (at 43.18 129.54 0)
+  (label "Emergency" (at 43.18 129.54 0)
     (effects (font (size 1.27 1.27)) (justify left bottom))
   )
@@
     (effects (font (size 1.27 1.27)) (justify left bottom))
   )
-  (label "Emergency_N" (at 44.45 101.6 0)
+  (label "Emergency" (at 44.45 101.6 0)
     (effects (font (size 1.27 1.27)) (justify left bottom))
   )
@@
     (effects (font (size 1.27 1.27)) (justify right bottom))
   )
-  (label "Emergency_P" (at 44.45 99.06 0)
-    (effects (font (size 1.27 1.27)) (justify left bottom))
-  )
   (label "JoyY" (at 43.18 137.16 0)
     (effects (font (size 1.27 1.27)) (justify left bottom))
@@
     (effects (font (size 1.27 1.27)) (justify left bottom))
   )
-  (label "Emergency_N" (at 43.18 132.08 0)
-    (effects (font (size 1.27 1.27)) (justify left bottom))
+  (symbol (lib_id "power:+3.3V") (at 43.18 132.08 270) (unit 1)
+    (in_bom yes) (on_board yes) (fields_autoplaced)
+    (property "Reference" "#PWR?" (id 0) (at 39.37 132.08 0)
+      (effects (font (size 1.27 1.27)) hide)
+    )
+    (property "Value" "+3.3V" (id 1) (at 46.355 132.5138 90)
+      (effects (font (size 1.27 1.27)) (justify left))
+    )
+    (property "Footprint" "" (id 2) (at 43.18 132.08 0)
+      (effects (font (size 1.27 1.27)) hide)
+    )
+    (property "Datasheet" "" (id 3) (at 43.18 132.08 0)
+      (effects (font (size 1.27 1.27)) hide)
+    )
+    (pin "1")
   )
   (symbol (lib_id "Connector:Conn_01x04_Male") (at 27.94 78.74 0) (unit 1)
@@
     (pin "1")
     (pin "2")
+  )
+  (symbol (lib_id "power:+3.3V") (at 44.45 99.06 270) (unit 1)
+    (in_bom yes) (on_board yes) (fields_autoplaced)
+    (property "Reference" "#PWR?" (id 0) (at 40.64 99.06 0)
+      (effects (font (size 1.27 1.27)) hide)
+    )
+    (property "Value" "+3.3V" (id 1) (at 47.625 99.4938 90)
+      (effects (font (size 1.27 1.27)) (justify left))
+    )
+    (property "Footprint" "" (id 2) (at 44.45 99.06 0)
+      (effects (font (size 1.27 1.27)) hide)
+    )
+    (property "Datasheet" "" (id 3) (at 44.45 99.06 0)
+      (effects (font (size 1.27 1.27)) hide)
+    )
+    (pin "1")
   )
   (symbol (lib_id "power:+5V") (at 44.45 81.28 270) (unit 1)
@@
   )
   (symbol_instances
+    (path "/24df4985-4b43-40d3-8f46-3158c91df2e5"
+      (reference "#PWR?") (unit 1) (value "+3.3V") (footprint "")
+    )
     (path "/411d2b70-0cea-425b-b95e-e0d5aa774241"
       (reference "#PWR?") (unit 1) (value "GND") (footprint "")
     )
+    (path "/6d008382-9155-4f6a-9cd8-94628c69bf8b"
+      (reference "#PWR?") (unit 1) (value "+3.3V") (footprint "")
+    )
     (path "/6e4c1c9d-d295-4d4f-8776-0ad5101d4b9d"
