File: catchrobo2023_OtherSubstrate/catchrobo2023_OtherSubstrate.kicad_pcb (KiCad board)
At the start: 2 copper layers, 72 x 47 mm, 12 parts, among them J1 Conn_01x02_Male, J2 Conn_01x02_Male, J3 Conn_01x02_Male, J4 Conn_01x02_Male, J5 Conn_01x04_Male, J6 Conn_01x04_Male, U1 STSPIN220, U2 STSPIN220

Commit message: MDを修正
Parts:
- removed J5, J6: Conn_01x04_Male, Connector_JST:JST_XH_S4B-XH-A-1_1x04_P2.50mm_Horizontal
- J1: value Conn_01x02_Male -> Conn_01x06_Male; footprint Connector_JST:JST_XH_S2B-XH-A-1_1x02_P2.50mm_Horizontal -> Connector_JST:JST_XH_S6B-XH-A_1x06_P2.50mm_Horizontal
- J3, J4: value Conn_01x02_Male -> Conn_01x04_Male; footprint Connector_JST:JST_XH_S2B-XH-A-1_1x02_P2.50mm_Horizontal -> Connector_JST:JST_XH_S4B-XH-A-1_1x04_P2.50mm_Horizontal
- moved J4 52.4 mm to (123.2, 106.8), turned to 180 degrees
- moved J3 33.5 mm to (97.2, 106.8), turned to 180 degrees
- moved J2 29.1 mm to (70.8, 120.2), turned to -90 degrees
- moved U1 26.5 mm to (93.5, 121.0)
- moved U2 25.5 mm to (119.5, 121.0)
- moved J1 22.1 mm to (97.8, 136.6)
Connections:
- J1 pad 1: Net-(J1-Pad1) -> +5V
- J1 pad 2: Net-(J1-Pad2) -> GND
- J2 pad 1: Net-(J2-Pad1) -> +7.5V
- J2 pad 2: Net-(J2-Pad2) -> GND
- J3 pad 1: +5V -> Net-(J3-Pad1)
- J3 pad 2: GND -> Net-(J3-Pad2)
- J4 pad 1: +7.5V -> Net-(J4-Pad1)
- J4 pad 2: GND -> Net-(J4-Pad2)
- U1 pad 11: Net-(J5-Pad1) -> Net-(J3-Pad1)
- U1 pad 12: Net-(J5-Pad2) -> Net-(J3-Pad2)
- U1 pad 13: Net-(J5-Pad3) -> Net-(J3-Pad3)
- U1 pad 14: Net-(J5-Pad4) -> Net-(J3-Pad4)
- U1 pad 7: Net-(J1-Pad2) -> /STEP1
- U1 pad 8: Net-(J1-Pad1) -> /DIR1
- U2 pad 11: Net-(J6-Pad1) -> Net-(J4-Pad1)
- U2 pad 12: Net-(J6-Pad2) -> Net-(J4-Pad2)
- U2 pad 13: Net-(J6-Pad3) -> Net-(J4-Pad3)
- U2 pad 14: Net-(J6-Pad4) -> Net-(J4-Pad4)
- U2 pad 7: Net-(J2-Pad2) -> /STEP2
- U2 pad 8: Net-(J2-Pad1) -> /DIR2
Routing:
- net /DIR2: track 0.00 -> 25.0 mm
- net /STEP2: track 0.00 -> 24.3 mm
- net +5V: track 69.8 -> 52.9 mm
- net Net-(J2-Pad1): track 13.6 -> 0.00 mm
- net Net-(J1-Pad1): track 13.6 -> 0.00 mm
- net Net-(J2-Pad2): track 11.5 -> 0.00 mm
- net Net-(J1-Pad2): track 11.5 -> 0.00 mm
- net /STEP1: track 0.00 -> 10.4 mm
- net /DIR1: track 0.00 -> 10.4 mm
- net Net-(J6-Pad1): track 8.94 -> 0.00 mm
- net Net-(J6-Pad2): track 8.92 -> 0.00 mm
- net Net-(J6-Pad3): track 8.91 -> 0.00 mm
- net Net-(J6-Pad4): track 8.89 -> 0.00 mm
- net Net-(J5-Pad1): track 8.79 -> 0.00 mm
- net Net-(J5-Pad2): track 8.77 -> 0.00 mm
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