File: catchrobo2023_OtherSubstrate/catchrobo2023_OtherSubstrate.kicad_sch (KiCad schematic)
At the start: 8 parts, among them J1 Conn_01x02_Male, J2 Conn_01x02_Male, J3 Conn_01x02_Male, J4 Conn_01x02_Male, J5 Conn_01x04_Male, J6 Conn_01x04_Male, U1 STSPIN220, U2 STSPIN220

Commit message: MDを修正
Parts:
- removed J1, J2, J3: Conn_01x02_Male, Connector_JST:JST_XH_S2B-XH-A-1_1x02_P2.50mm_Horizontal, symbol Connector:Conn_01x02_Male
- added J1: Conn_01x06_Male, Connector_JST:JST_XH_S6B-XH-A_1x06_P2.50mm_Horizontal, symbol Connector:Conn_01x06_Male
- renumbered J4 to J2, J5 to J3, J6 to J4
Connections:
- net +5V: now also J1.1 (Pin_1)
- net GND: now also J1.2 (Pin_2)
- net STEP2: now reaches U2.7 (STEP/MODE3)
- net STEP2: now also J1.5 (Pin_5)
- net DIR2: now reaches U2.8 (DIR/MODE4)
- net DIR2: now also J1.6 (Pin_6)
- net DIR1: now reaches U1.8 (DIR/MODE4)
- net DIR1: now also J1.4 (Pin_4)
- net STEP1: now reaches U1.7 (STEP/MODE3)
- net STEP1: now also J1.3 (Pin_3)
